File: shields/cnc/cnc.kicad_pcb (KiCad board)
At the start: 2 copper layers, 68.6 x 53.3 mm, 44 parts, among them J1 Conn_01x02_Male, J10 Conn_01x02_Male, J11 Conn_01x02_Male, J12 Conn_01x02_Male, J13 Conn_01x03_Male, J14 Conn_01x03_Male, J15 Conn_01x03_Male, J16 Conn_01x03_Male, J17 Conn_01x03_Male, J18 Conn_01x03_Male, J19 Conn_01x02_Male, J2 Conn_01x02_Male, J20 Conn_01x03_Male, J21 Conn_01x03_Male, J22 Conn_01x03_Male, J23 Conn_01x02_Male, J24 Conn_01x02_Male, J3 Conn_01x02_Male, J4 Conn_01x02_Male, J5 Conn_01x02_Male, J6 Conn_01x02_Male, J7 Conn_01x02_Male, J8 Conn_01x02_Male, J9 Conn_01x02_Male, P1 Power, P2 Analog, P3 Digital, P4 Digital, P5 CONN_01X01, P6 CONN_01X01, P7 CONN_01X01, P8 CONN_01X01, Q1 IRF540N, Q2 IRF540N, U1 4N25, U2 4N25

Commit message: placa pronta
Parts:
- added HS1: Heatsink, Heatsink:Heatsink_Fischer_SK104-STC-STIC_35x13mm_2xDrill2.5mm, F.Cu at (130.7, 125.7)
- added HS2: Heatsink, Heatsink:Heatsink_Fischer_SK104-STC-STIC_35x13mm_2xDrill2.5mm, F.Cu at (189.7, 127.0)
- J19: footprint Connector_Molex:Molex_KK-254_AE-6410-03A_1x03_P2.54mm_Vertical -> Connector_Molex:Molex_KK-254_AE-6410-02A_1x02_P2.54mm_Vertical
- moved J10 117.8 mm to (152.9, 40.6), turned to 180 degrees
- moved J9 112.9 mm to (159.3, 40.6), turned to 180 degrees
- moved J6 111.7 mm to (128.1, 82.5), turned to 270 degrees
- moved J8 105.0 mm to (165.6, 40.6), turned to 180 degrees
- moved J3 100.0 mm to (152.9, 47.6), turned to 180 degrees
- moved J2 99.6 mm to (159.3, 47.6), turned to 180 degrees
- moved J4 99.5 mm to (140.2, 73.0)
- moved J1 95.8 mm to (165.6, 47.6), turned to 180 degrees
- moved J12 85.1 mm to (164.3, 94.6)
- moved J5 84.8 mm to (156.7, 94.6)
- moved J15 83.9 mm to (159.3, 81.6), turned to 270 degrees
- moved J16 82.8 mm to (159.3, 71.5), turned to 270 degrees
- moved J20 82.6 mm to (159.3, 61.3), turned to 270 degrees
- moved J21 78.6 mm to (168.2, 61.3), turned to 270 degrees
- moved Q1 71.3 mm to (135.1, 127.6), turned to 90 degrees
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Connections:
- P2 pad 5: /A4(SDA) -> /A4(SDA)1
- P2 pad 6: /A5(SCL) -> /A5(SCL)1
- R2 pad 1: Net-(R2-Pad1) -> Net-(Q1-Pad1)
- R2 pad 2: +24V -> Net-(R2-Pad2)
- R3 pad 2: Net-(R2-Pad1) -> GNDPWR
- R5 pad 1: Net-(R5-Pad1) -> Net-(Q2-Pad1)
- R5 pad 2: +24V -> Net-(R5-Pad2)
- R6 pad 2: Net-(R5-Pad1) -> GNDPWR
- U1 pad 4: GNDPWR -> Net-(R2-Pad2)
- U1 pad 5: Net-(R2-Pad1) -> +24V
- U2 pad 4: GNDPWR -> Net-(R5-Pad2)
- U2 pad 5: Net-(R5-Pad1) -> +24V
Routing:
- net GND: track 0.00 -> 339.8 mm, vias 0 -> 4
- net +5V: track 0.00 -> 157.5 mm, vias 0 -> 6
- net GNDPWR: track 0.00 -> 110.9 mm
- net +24V: track 0.00 -> 75.5 mm, vias 0 -> 2
- net Enable: track 0.00 -> 61.0 mm
- net SpinDir: track 0.00 -> 38.8 mm
- net Net-(J4-Pad1): track 0.00 -> 37.8 mm
- net Step-X: track 0.00 -> 36.3 mm
- net Dir-X: track 0.00 -> 34.0 mm
- net Net-(Q1-Pad1): track 0.00 -> 29.0 mm
- net Step-Y: track 0.00 -> 26.5 mm
- net SpinEnable: track 0.00 -> 24.2 mm
- net Dir-Y: track 0.00 -> 22.8 mm
- net Net-(D1-Pad1): track 0.00 -> 22.4 mm
- net Net-(D2-Pad1): track 0.00 -> 21.1 mm
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- added copper zone on B.Cu, net GND
- added copper zone on F.Cu, net GND
- added copper zone on B.Cu, net GNDPWR
- added copper zone on F.Cu, net GNDPWR
Other:
- board size 68.6 x 53.3 mm -> 73 x 110.5 mm
- net class 24 added: clearance 0.3048, trace_width 3.048, via_dia 1.5, via_drill 0.6
- net class Default: clearance 0.2 -> 0.3048; trace_width 0.25 -> 0.8; via_dia 0.6 -> 1.5; via_drill 0.4 -> 0.6
- rule trace_clearance: 0.2 -> 0.3048
- rule trace_min: 0.2 -> 0.6096
