File: shields/cnc/cnc.sch (KiCad schematic (older format))
At the start: 44 parts, among them J1 Conn_01x02_Male, J10 Conn_01x02_Male, J11 Conn_01x02_Male, J12 Conn_01x02_Male, J13 Conn_01x03_Male, J14 Conn_01x03_Male, J15 Conn_01x03_Male, J16 Conn_01x03_Male, J17 Conn_01x03_Male, J18 Conn_01x03_Male, J19 Conn_01x02_Male, J2 Conn_01x02_Male, J20 Conn_01x03_Male, J21 Conn_01x03_Male, J22 Conn_01x03_Male, J23 Conn_01x02_Male, J24 Conn_01x02_Male, J3 Conn_01x02_Male, J4 Conn_01x02_Male, J5 Conn_01x02_Male, J6 Conn_01x02_Male, J7 Conn_01x02_Male, J8 Conn_01x02_Male, J9 Conn_01x02_Male, P1 Power, P2 Analog, P3 Digital, P4 Digital, P5 CONN_01X01, P6 CONN_01X01, P7 CONN_01X01, P8 CONN_01X01, Q1 IRF540N, Q2 IRF540N, U1 4N25, U2 4N25

Commit message: placa pronta
Parts:
- added HS1, HS2: Heatsink, Heatsink:Heatsink_Fischer_SK104-STC-STIC_35x13mm_2xDrill2.5mm, symbol Mechanical:Heatsink
- J19: footprint Connector_Molex:Molex_KK-254_AE-6410-03A_1x03_P2.54mm_Vertical -> Connector_Molex:Molex_KK-254_AE-6410-02A_1x02_P2.54mm_Vertical
Connections:
- net +24V: now also U1.5, U2.5; no longer R2.2, R5.2
- net A4(SDA): no longer P2.5 (Pin_5)
- net A5(SCL): no longer P2.6 (Pin_6)
- net GNDPWR: now also R3.2, R6.2; no longer U1.4, U2.4
- net at Q1.1 (G), R3.1: now also R2.1
- net at Q2.1 (G), R6.1: now also R5.1
- new net: R2.2, U1.4
- new net: R5.2, U2.4
- new net A4(SDA)1: P2.5 (Pin_5)
- new net A5(SCL)1: P2.6 (Pin_6)
Other:
- moved on the sheet: D1, D2, J11, J12, J19, J23, J24, J4, J7, Q1, Q2, R1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
